File: hardware/dual_button.kicad_pcb (KiCad board)
At the start: 2 copper layers, 20 x 45 mm, 25 parts, among them P1 CON-SENSOR2, P2 DEBUG, P3 BOOT, SW1 TACT_SWITCH_12MM, SW2 TACT_SWITCH_12MM, U1 XMC1XXX24, U2 DRILL, U3 DRILL, U4 DRILL, U5 DRILL

Commit message: change drilling holes to new standard
Parts:
- U2, U3, U4, U5: footprint DRILL_NP -> kicad-libraries:DRILL_NP
