File: hardware/dual-button-v2.kicad_pcb (KiCad board)
At the start: 2 copper layers, 20 x 45 mm, 25 parts, among them P1 CON-SENSOR2, P2 DEBUG, P3 BOOT, SW1 TACT_SWITCH_12MM, SW2 TACT_SWITCH_12MM, U1 XMC1XXX24, U2 DRILL, U3 DRILL, U4 DRILL, U5 DRILL

Commit message: fix logo position, fix origin
Parts:
- Fiducial_Mark (x2): footprint Fiducial_Mark -> kicad-libraries:Fiducial_Mark
- moved G*** 1.40 mm to (169.0, 109.0)
Changed lines of the file:
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@@
-(kicad_pcb (version 4) (host pcbnew 4.0.7-e2-6376~58~ubuntu17.04.1)
+(kicad_pcb (version 4) (host pcbnew 4.0.7-e2-6376~61~ubuntu18.04.1)
   (general
     (links 47)
     (no_connects 0)
-    (area 15.21415 86.309499 179.4 195.930793)
+    (area 15.21415 85.644999 179.855001 195.930793)
     (thickness 1.6002)
     (drawings 16)
@@
   (layers
     (0 Vorderseite signal)
-    (31 Rückseite signal)
+    (31 Rückseite signal hide)
     (32 B.Adhes user)
     (33 F.Adhes user)
@@
     (pad_drill 1.6)
     (pad_to_mask_clearance 0)
-    (aux_axis_origin 159.1 131.4)
-    (grid_origin 159.1 131.4)
+    (aux_axis_origin 159 86.5)
+    (grid_origin 159 86.5)
     (visible_elements FFFFFFBF)
     (pcbplotparams
@@
       (xy 3.1242 3.1242)) (layer F.SilkS) (width 0.00254))
   )
-  (module Fiducial_Mark (layer Vorderseite)
-    (at 160.5 93)
-    (path Fiducial_Mark)
-    (attr smd)
-    (fp_text reference Fiducial_Mark (at 0 0) (layer F.SilkS) hide
-      (effects (font (size 0.127 0.127) (thickness 0.03302)))
-    )
-    (fp_text value VAL** (at 0 -0.29972) (layer F.SilkS) hide
-      (effects (font (size 0.127 0.127) (thickness 0.03302)))
-    )
-    (fp_circle (center 0 0) (end 1.15062 0) (layer Dwgs.User) (width 0.01016))
-    (pad 1 smd circle (at 0 0) (size 1.00076 1.00076) (layers Vorderseite F.Mask)
-      (clearance 0.65024))
-  )
-  (module Fiducial_Mark (layer Vorderseite)
-    (at 177.5 117)
-    (path Fiducial_Mark)
-    (attr smd)
-    (fp_text reference Fiducial_Mark (at 0 0) (layer F.SilkS) hide
-      (effects (font (size 0.127 0.127) (thickness 0.03302)))
-    )
-    (fp_text value VAL** (at 0 -0.29972) (layer F.SilkS) hide
-      (effects (font (size 0.127 0.127) (thickness 0.03302)))
-    )
-    (fp_circle (center 0 0) (end 1.15062 0) (layer Dwgs.User) (width 0.01016))
-    (pad 1 smd circle (at 0 0) (size 1.00076 1.00076) (layers Vorderseite F.Mask)
-      (clearance 0.65024))
-  )
   (module kicad-libraries:TACT_SWITCH_12mm (layer Vorderseite)
     (at 169 121.5 315)
@@
   )
   (module kicad-libraries:WEEE_7mm (layer Rückseite)
-    (at 169 121.49 90)
+    (at 169 121.5 90)
     (fp_text reference VAL (at 0 0 90) (layer B.SilkS) hide
       (effects (font (size 0.2 0.2) (thickness 0.05)) (justify mirror))
@@
   )
   (module kicad-libraries:Logo_CoMCU (layer Rückseite)
-    (at 169 107.6 90)
+    (at 169 109 90)
     (fp_text reference G*** (at 0 0 90) (layer B.SilkS) hide
       (effects (font (thickness 0.3)) (justify mirror))
@@
       (clearance 0.89916))
   )
+  (module kicad-libraries:Fiducial_Mark (layer Vorderseite)
+    (at 160.5 93)
+    (path Fiducial_Mark)
+    (attr smd)
+    (fp_text reference Fiducial_Mark (at 0 0) (layer F.SilkS) hide
+      (effects (font (size 0.127 0.127) (thickness 0.03302)))
+    )
+    (fp_text value VAL** (at 0 -0.29972) (layer F.SilkS) hide
+      (effects (font (size 0.127 0.127) (thickness 0.03302)))
+    )
+    (fp_circle (center 0 0) (end 1.15062 0) (layer Dwgs.User) (width 0.01016))
+    (pad 1 smd circle (at 0 0) (size 1.00076 1.00076) (layers Vorderseite F.Paste F.Mask)
+      (clearance 0.65024))
+  )
+  (module kicad-libraries:Fiducial_Mark (layer Vorderseite)
+    (at 177.5 117)
+    (path Fiducial_Mark)
+    (attr smd)
+    (fp_text reference Fiducial_Mark (at 0 0) (layer F.SilkS) hide
+      (effects (font (size 0.127 0.127) (thickness 0.03302)))
+    )
+    (fp_text value VAL** (at 0 -0.29972) (layer F.SilkS) hide
+      (effects (font (size 0.127 0.127) (thickness 0.03302)))
+    )
+    (fp_circle (center 0 0) (end 1.15062 0) (layer Dwgs.User) (width 0.01016))
+    (pad 1 smd circle (at 0 0) (size 1.00076 1.00076) (layers Vorderseite F.Paste F.Mask)
+      (clearance 0.65024))
+  )
   (gr_text Status (at 177.31 99.1 270) (layer F.SilkS)
