File: hardware/dual-button-v2.kicad_pcb (KiCad board)
At the start: 2 copper layers, 20 x 45 mm, 25 parts, among them P1 CON-SENSOR2, P2 DEBUG, P3 BOOT, SW1 TACT_SWITCH_12MM, SW2 TACT_SWITCH_12MM, U1 XMC1XXX24, U2 DRILL, U3 DRILL, U4 DRILL, U5 DRILL

Commit message: Change capacitor footprint(s) to C0402F
Parts:
- C2: footprint kicad-libraries:C0402E -> kicad-libraries:C0402F
Changed lines of the file:
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@@
-(kicad_pcb (version 4) (host pcbnew 4.0.7-e2-6376~61~ubuntu18.04.1)
+(kicad_pcb (version 4) (host pcbnew 4.0.2+dfsg1-stable)
   (general
     (links 47)
     (no_connects 0)
-    (area 15.21415 85.644999 179.855001 195.930793)
+    (area 158.809499 86.309499 179.190501 131.691001)
     (thickness 1.6002)
     (drawings 16)
@@
   )
   (setup
-    (last_trace_width 0.29972)
+    (last_trace_width 0.55)
     (user_trace_width 0.2)
     (user_trace_width 0.25)
@@
       (xy 2.48217 3.513666) (xy 2.482863 3.409859) (xy 2.482863 3.409859)) (layer B.SilkS) (width 0.1))
   )
-  (module kicad-libraries:C0402E (layer Vorderseite)
-    (at 172.6 104.9 270)
-    (attr smd)
-    (fp_text reference C2 (at 0 0.125 270) (layer F.Fab)
-      (effects (font (size 0.2 0.2) (thickness 0.05)))
-    )
-    (fp_text value 220pF (at 0 -0.275 270) (layer F.Fab)
-      (effects (font (size 0.2 0.2) (thickness 0.05)))
-    )
-    (fp_line (start -0.8509 -0.44958) (end 0.8509 -0.44958) (layer F.Fab) (width 0.001))
-    (fp_line (start 0.8509 -0.44958) (end 0.8509 0.44958) (layer F.Fab) (width 0.001))
-    (fp_line (start 0.8509 0.44958) (end -0.8509 0.44958) (layer F.Fab) (width 0.001))
-    (fp_line (start -0.8509 0.44958) (end -0.8509 -0.44958) (layer F.Fab) (width 0.001))
-    (pad 1 smd rect (at -0.65 0 270) (size 0.7 0.9) (layers Vorderseite F.Paste F.Mask)
-      (net 3 GND))
-    (pad 2 smd rect (at 0.65 0 270) (size 0.7 0.9) (layers Vorderseite F.Paste F.Mask)
-      (net 7 "Net-(C2-Pad2)"))
-    (model Capacitors_SMD/C_0402.wrl
-      (at (xyz 0 0 0))
-      (scale (xyz 1 1 1))
-      (rotate (xyz 0 0 0))
-    )
-  )
   (module kicad-libraries:D0603F (layer Vorderseite)
     (at 177.26 101.54 180)
@@
       (clearance 0.65024))
   )
+  (module kicad-libraries:C0402F (layer Vorderseite)
+    (at 172.6 104.9 270)
+    (fp_text reference C2 (at 0.1 0.15 270) (layer F.Fab)
+      (effects (font (size 0.2 0.2) (thickness 0.05)))
+    )
+    (fp_text value 220pF (at 0 -0.15 270) (layer F.Fab)
+      (effects (font (size 0.2 0.2) (thickness 0.05)))
+    )
+    (fp_line (start -0.9 -0.45) (end 0.9 -0.45) (layer F.Fab) (width 0.025))
+    (fp_line (start 0.9 -0.45) (end 0.9 0.45) (layer F.Fab) (width 0.025))
+    (fp_line (start 0.9 0.45) (end -0.9 0.45) (layer F.Fab) (width 0.025))
+    (fp_line (start -0.9 0.45) (end -0.9 -0.45) (layer F.Fab) (width 0.025))
+    (pad 2 smd rect (at 0.5 0 270) (size 0.6 0.7) (layers Vorderseite F.Paste F.Mask)
+      (net 7 "Net-(C2-Pad2)"))
+    (pad 1 smd rect (at -0.5 0 270) (size 0.6 0.7) (layers Vorderseite F.Paste F.Mask)
+      (net 3 GND))
+    (model Capacitors_SMD/C_0402.wrl
+      (at (xyz 0 0 0))
+      (scale (xyz 1 1 1))
+      (rotate (xyz 0 0 0))
+    )
+  )
   (gr_text Status (at 177.31 99.1 270) (layer F.SilkS)
     (effects (font (size 0.75 0.75) (thickness 0.15)))
@@
   (segment (start 168.98 106.11) (end 169.45 106.11) (width 0.2) (layer Vorderseite) (net 2))
   (segment (start 169.45 106.11) (end 169.85967 105.70033) (width 0.2) (layer Vorderseite) (net 2))
+  (segment (start 172.6 104.4) (end 173.23 104.4) (width 0.55) (layer Vorderseite) (net 3))
+  (via (at 173.23 104.4) (size 0.55) (drill 0.25) (layers Vorderseite Rückseite) (net 3))
   (segment (start 167.033553 112.543553) (end 167.38 112.89) (width 0.2) (layer Vorderseite) (net 3))
   (via (at 167.38 112.89) (size 0.55) (drill 0.25) (layers Vorderseite Rückseite) (net 3))
@@
   (segment (start 177.8 103.1) (end 177.8 104.08) (width 0.55) (layer Vorderseite) (net 3))
   (via (at 177.8 104.08) (size 0.55) (drill 0.25) (layers Vorderseite Rückseite) (net 3))
-  (segment (start 172.6 104.25) (end 172.6 103.62) (width 0.55) (layer Vorderseite) (net 3))
-  (via (at 172.6 103.62) (size 0.55) (drill 0.25) (layers Vorderseite Rückseite) (net 3))
   (via (at 171.26 112.9) (size 0.55) (drill 0.25) (layers Vorderseite Rückseite) (net 3))
   (segment (start 170.26 112) (end 170.82 112) (width 0.55) (layer Vorderseite) (net 3))
@@
   (segment (start 174.4 110.25) (end 172.50076 110.25) (width 0.55) (layer Vorderseite) (net 6))
   (segment (start 172.50076 110.25) (end 172.46 110.20924) (width 0.45) (layer Vorderseite) (net 6))
+  (segment (start 174.4 105.25) (end 173.22 105.25) (width 0.2) (layer Vorderseite) (net 7))
+  (segment (start 173.07 105.4) (end 172.6 105.4) (width 0.2) (layer Vorderseite) (net 7))
+  (segment (start 173.22 105.25) (end 173.07 105.4) (width 0.2) (layer Vorderseite) (net 7))
   (segment (start 172.6 105.55) (end 172.6 106.2757) (width 0.2) (layer Vorderseite) (net 7))
   (segment (start 172.6 106.2757) (end 172.675 106.3507) (width 0.2) (layer Vorderseite) (net 7))
-  (segment (start 174.4 105.25) (end 173.44 105.25) (width 0.2) (layer Vorderseite) (net 7))
-  (segment (start 173.14 105.55) (end 172.6 105.55) (width 0.2) (layer Vorderseite) (net 7))
-  (segment (start 173.44 105.25) (end 173.14 105.55) (width 0.2) (layer Vorderseite) (net 7))
   (segment (start 174.81033 101.84967) (end 174.86033 101.84967) (width 0.3) (layer Vorderseite) (net 8))
   (segment (start 174.86033 101.84967) (end 175.17 101.54) (width 0.25) (layer Vorderseite) (net 8))
