File: hardware/dual-button-v2.kicad_pcb (KiCad board)
At the start: 2 copper layers, 20 x 45 mm, 25 parts, among them P1 CON-SENSOR2, P2 DEBUG, P3 BOOT, SW1 TACT_SWITCH_12MM, SW2 TACT_SWITCH_12MM, U1 XMC1XXX24, U2 DRILL, U3 DRILL, U4 DRILL, U5 DRILL

Commit message: specify processor
Parts:
- U1: value XMC1XXX24 -> XMC11XX24
Changed lines of the file:
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@@
-(kicad_pcb (version 4) (host pcbnew 4.0.2+dfsg1-stable)
+(kicad_pcb (version 4) (host pcbnew 4.0.7-e2-6376~61~ubuntu18.04.1)
   (general
     (links 47)
     (no_connects 0)
-    (area 158.809499 86.309499 179.190501 131.691001)
+    (area 15.21415 85.644999 179.855001 195.930793)
     (thickness 1.6002)
     (drawings 16)
@@
       (effects (font (size 0.3 0.3) (thickness 0.075)))
     )
-    (fp_text value XMC1XXX24 (at 0 0.8 225) (layer F.Fab)
+    (fp_text value XMC11XX24 (at 0 0.8 225) (layer F.Fab)
       (effects (font (size 0.3 0.3) (thickness 0.075)))
     )

Commit message: specify processor
Parts:
- U1: value XMC11XX24 -> XMC1100
